File: hardware/motorpcb i think/motorpcb i think.kicad_pcb (KiCad board)
At the start: 2 copper layers, 6.5 x 0.7 mm, 36 parts, among them J1 USB_C_Receptacle_USB2.0_16P, J10 Conn_01x04_Pin, J11 Conn_01x02_Pin, J2 USB_C_Receptacle_USB2.0_16P, J3 Conn_01x15_Pin, J4 Screw_Terminal_01x02, J5 Screw_Terminal_01x02, J6 Conn_01x15_Pin, J7 Conn_01x04_Pin, J8 Conn_01x04_Pin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

Commit message: schematic finished
Parts:
- added +3V3: TestPoint, TestPoint:TestPoint_Keystone_5010-5014_Multipurpose, F.Cu at (90.0, 20.9)
- added J12: Screw_Terminal_01x02, TerminalBlock:TerminalBlock_MaiXu_MX126-5.0-02P_1x02_P5.00mm, F.Cu at (96.5, 23.4)
- added T1: GND, TestPoint:TestPoint_Keystone_5010-5014_Multipurpose, F.Cu at (90.0, 25.9)
- added T2: VHV, TestPoint:TestPoint_Keystone_5010-5014_Multipurpose, F.Cu at (90.0, 30.9)
- added T3: M+, TestPoint:TestPoint_Keystone_5010-5014_Multipurpose, F.Cu at (90.0, 36.0)
Connections:
- C6 pad 1: +12V -> /VHV
- J2 pad A1B12: GND -> (no net)
- J2 pad A4B9: +12V -> (no net)
- J2 pad B1A12: GND -> (no net)
- J2 pad B4A9: +12V -> (no net)
- U3 pad 1: +12V -> /VHV
- U3 pad 8: +12V -> /VHV
